Commit message: Update dsr.ros2_control.xacro

File: dsr_moveit2/m1013_moveit_config/config/dsr.ros2_control.xacro (robot description, xacro)
@@ -61,4 +61,13 @@
                 </state_interface>
             </joint>
+            <joint name="finger_joint">
+                <command_interface name="position"/>
+                <state_interface name="position">
+                  <!-- <param name="initial_value">${initial_positions['finger_joint']}</param> -->
+                </state_interface>
+                <state_interface name="velocity">
+                    <param name="initial_value">0.0</param>
+                </state_interface>
+            </joint>
         </ros2_control>
     </xacro:macro>
