Commit message: Update onrobot_rg6_model_macro.xacro

File: onrobot/onrobot_rg_description/urdf/onrobot_rg6_model_macro.xacro (robot description, xacro)
@@ -11,9 +11,9 @@
       </inertial>
       <visual>
-        <origin xyz="0 0 0" rpy="0 0 0" />
+        <origin xyz="0 0 0" rpy="0 0 0" /
         <geometry>
-          <mesh filename="package://onrobot_rg_description/meshes/rg6/visual/outer_knuckle.stl" />
+          <mesh filename="package://dsr_description2/meshes/rg6/collision/outer_knuckle.stl" />
         </geometry>
-        <material name="">
+        <material name=""
           <color rgba="0.8 0.8 0.8 1" />
         </material>
@@ -22,6 +22,6 @@
         <origin xyz="0 0 0" rpy="0 0 0" />
         <geometry>
-          <mesh filename="package://onrobot_rg_description/meshes/rg6/collision/outer_knuckle.stl" />
-        </geometry>
+          <mesh filename="package://dsr_description2/meshes/rg6/collision/outer_knuckle.stl" />
+        </geometry
       </collision>
     </link>
@@ -33,5 +33,5 @@
     </gazebo>
   </xacro:macro>
-  <xacro:macro name="inner_knuckle" params="prefix fingerprefix">
+  <xacro:macro name="inner_knuckle" params="prefix fingerprefix"
     <link name="${prefix}${fingerprefix}_inner_knuckle">
       <inertial>
@@ -43,6 +43,5 @@
         <origin xyz="0 0 0" rpy="0 0 0" />
         <geometry>
-          <mesh filename="package://onrobot_rg_description/meshes/rg6/visual/inner_knuckle.stl" />
-        </geometry>
+          <mesh filename="package://dsr_description2/meshes/rg6/visual/inner_knuckle.stl" />        </geometry>
         <material name="">
           <color rgba="0.8 0.8 0.8 1" />
@@ -52,5 +51,5 @@
         <origin xyz="0 0 0" rpy="0 0 0" />
         <geometry>
-          <mesh filename="package://onrobot_rg_description/meshes/rg6/collision/inner_knuckle.stl" />
+          <mesh filename="package://dsr_description2/meshes/rg6/collision/inner_knuckle.stl" />
         </geometry>
       </collision>
@@ -65,26 +64,26 @@
   <xacro:macro name="inner_finger" params="prefix fingerprefix">
     <link name="${prefix}${fingerprefix}_inner_finger">
-      <inertial>
+      <inertial
         <origin xyz="0.0 0.0 0.0" rpy="0 0 0" />
-        <mass value="0.05" />
+        <mass value="0.05" /
         <inertia ixx="1.0E-03" ixy="1.0E-06" ixz="1.0E-06" iyy="1.0E-03" iyz="1.0E-06" izz="1.0E-03" />
-      </inertial>
+      </inertial
       <visual>
         <origin xyz="0 0 0" rpy="0 0 0" />
         <geometry>
-          <mesh filename="package://onrobot_rg_description/meshes/rg6/visual/inner_finger.stl" />
+          <mesh filename="package://dsr_description2/meshes/rg6/visual/inner_finger.stl" /
         </geometry>
-        <material name="">
-          <color rgba="0.1 0.1 0.1 1" />
+        <material name=""
+          <color rgba="0.1 0.1 0.1 1" /
         </material>
       </visual>
-      <collision>
+      <collision
         <origin xyz="0 0 0" rpy="0 0 0" />
         <geometry>
-          <mesh filename="package://onrobot_rg_description/meshes/rg6/collision/inner_finger.stl" />
+          <mesh filename="package://dsr_description2/meshes/rg6/collision/inner_finger.stl" />
         </geometry>
       </collision>
     </link>
-    <gazebo reference="${prefix}${fingerprefix}_inner_finger">
+    <gazebo reference="${prefix}${fingerprefix}_inner_finger"
       <kp>1000000.0</kp>
       <kd>1.0</kd>
@@ -123,5 +122,5 @@
       <child link="${prefix}left_outer_knuckle" />
       <axis xyz="-1 0 0" />
-      <limit lower="-0.628319" upper="0.628319" velocity="2.0" effort="1000" />
+      <limit lower="-0.628319" upper="0.628319" velocity="2.0" effort="1000" /
     </joint>
     <xacro:finger_joints prefix="${prefix}" fingerprefix="left" reflect="1.0"/>

Commit message: Update onrobot_rg6_model_macro.xacro

File: onrobot/onrobot_rg_description/urdf/onrobot_rg6_model_macro.xacro (robot description, xacro)
@@ -11,9 +11,9 @@
       </inertial>
       <visual>
-        <origin xyz="0 0 0" rpy="0 0 0" /
+        <origin xyz="0 0 0" rpy="0 0 0" />
         <geometry>
           <mesh filename="package://dsr_description2/meshes/rg6/collision/outer_knuckle.stl" />
         </geometry>
-        <material name=""
+        <material name="">
           <color rgba="0.8 0.8 0.8 1" />
         </material>
@@ -23,5 +23,5 @@
         <geometry>
           <mesh filename="package://dsr_description2/meshes/rg6/collision/outer_knuckle.stl" />
-        </geometry
+        </geometry>
       </collision>
     </link>
@@ -33,5 +33,5 @@
     </gazebo>
   </xacro:macro>
-  <xacro:macro name="inner_knuckle" params="prefix fingerprefix"
+  <xacro:macro name="inner_knuckle" params="prefix fingerprefix">
     <link name="${prefix}${fingerprefix}_inner_knuckle">
       <inertial>
@@ -64,19 +64,19 @@
   <xacro:macro name="inner_finger" params="prefix fingerprefix">
     <link name="${prefix}${fingerprefix}_inner_finger">
-      <inertial
+      <inertial>
         <origin xyz="0.0 0.0 0.0" rpy="0 0 0" />
-        <mass value="0.05" /
+        <mass value="0.05" />
         <inertia ixx="1.0E-03" ixy="1.0E-06" ixz="1.0E-06" iyy="1.0E-03" iyz="1.0E-06" izz="1.0E-03" />
-      </inertial
+      </inertial>
       <visual>
         <origin xyz="0 0 0" rpy="0 0 0" />
         <geometry>
-          <mesh filename="package://dsr_description2/meshes/rg6/visual/inner_finger.stl" /
+          <mesh filename="package://dsr_description2/meshes/rg6/visual/inner_finger.stl" />
         </geometry>
-        <material name=""
-          <color rgba="0.1 0.1 0.1 1" /
+        <material name="">
+          <color rgba="0.1 0.1 0.1 1" />
         </material>
       </visual>
-      <collision
+      <collision>
         <origin xyz="0 0 0" rpy="0 0 0" />
         <geometry>
@@ -85,5 +85,5 @@
       </collision>
     </link>
-    <gazebo reference="${prefix}${fingerprefix}_inner_finger"
+    <gazebo reference="${prefix}${fingerprefix}_inner_finger">
       <kp>1000000.0</kp>
       <kd>1.0</kd>
@@ -122,5 +122,5 @@
       <child link="${prefix}left_outer_knuckle" />
       <axis xyz="-1 0 0" />
-      <limit lower="-0.628319" upper="0.628319" velocity="2.0" effort="1000" /
+      <limit lower="-0.628319" upper="0.628319" velocity="2.0" effort="1000" />
     </joint>
     <xacro:finger_joints prefix="${prefix}" fingerprefix="left" reflect="1.0"/>

Commit message: Update onrobot_rg6_model_macro.xacro

File: onrobot/onrobot_rg_description/urdf/onrobot_rg6_model_macro.xacro (robot description, xacro)
@@ -13,5 +13,5 @@
         <origin xyz="0 0 0" rpy="0 0 0" />
         <geometry>
-          <mesh filename="package://onrobot_rg_description/meshes/rg6/visual/outer_knuckle.stl" />
+          <mesh filename="package://dsr_description2/meshes/rg6/visual/outer_knuckle.stl" />
         </geometry>
         <material name="">
@@ -22,5 +22,5 @@
         <origin xyz="0 0 0" rpy="0 0 0" />
         <geometry>
-          <mesh filename="package://onrobot_rg_description/meshes/rg6/collision/outer_knuckle.stl" />
+          <mesh filename="package://dsr_description2/meshes/rg6/collision/outer_knuckle.stl" />
         </geometry>
       </collision>
@@ -43,5 +43,5 @@
         <origin xyz="0 0 0" rpy="0 0 0" />
         <geometry>
-          <mesh filename="package://onrobot_rg_description/meshes/rg6/visual/inner_knuckle.stl" />
+          <mesh filename="package://dsr_description2/meshes/rg6/visual/inner_knuckle.stl" />
         </geometry>
         <material name="">
@@ -52,5 +52,5 @@
         <origin xyz="0 0 0" rpy="0 0 0" />
         <geometry>
-          <mesh filename="package://onrobot_rg_description/meshes/rg6/collision/inner_knuckle.stl" />
+          <mesh filename="package://dsr_description2/meshes/rg6/collision/inner_knuckle.stl" />
         </geometry>
       </collision>
@@ -73,5 +73,5 @@
         <origin xyz="0 0 0" rpy="0 0 0" />
         <geometry>
-          <mesh filename="package://onrobot_rg_description/meshes/rg6/visual/inner_finger.stl" />
+          <mesh filename="package://dsr_description2/meshes/rg6/visual/inner_finger.stl" />
         </geometry>
         <material name="">
@@ -82,5 +82,5 @@
         <origin xyz="0 0 0" rpy="0 0 0" />
         <geometry>
-          <mesh filename="package://onrobot_rg_description/meshes/rg6/collision/inner_finger.stl" />
+          <mesh filename="package://dsr_description2/meshes/rg6/collision/inner_finger.stl" />
         </geometry>
       </collision>
