Commit message: Update onrobot_rg6.xacro

File: onrobot/onrobot_rg_description/urdf/onrobot_rg6.xacro (robot description, xacro)
@@ -1,5 +1,5 @@
 <?xml version="1.0"?>
 <robot xmlns:xacro="http://ros.org/wiki/xacro">
-  <xacro:macro name="onrobot_rg6_base_link" params="prefix">
+  <xacro:macro name="onrobot_rg6_base_link" params="prefix"
     <link name="${prefix}onrobot_rg6_base_link">
       <inertial>
@@ -11,5 +11,5 @@
         <origin xyz="0 0 0" rpy="0 0 0" />
         <geometry>
-          <mesh filename="package://onrobot_rg_description/meshes/rg6/visual/base_link.stl" />
+          <mesh filename="package://dsr_description2/meshes/rg6/visual/base_link.stl" /
         </geometry>
         <material name="">
@@ -19,6 +19,6 @@
       <collision>
         <origin xyz="0 0 0" rpy="0 0 0" />
-        <geometry>
-          <mesh filename="package://onrobot_rg_description/meshes/rg6/collision/base_link.stl" />
+        <geometry
+          <mesh filename="package://dsr_description2/meshes/rg6/collision/base_link.stl" />
         </geometry>
       </collision>

Commit message: Update onrobot_rg6.xacro

File: onrobot/onrobot_rg_description/urdf/onrobot_rg6.xacro (robot description, xacro)
@@ -1,5 +1,5 @@
 <?xml version="1.0"?>
 <robot xmlns:xacro="http://ros.org/wiki/xacro">
-  <xacro:macro name="onrobot_rg6_base_link" params="prefix"
+  <xacro:macro name="onrobot_rg6_base_link" params="prefix">
     <link name="${prefix}onrobot_rg6_base_link">
       <inertial>
@@ -11,5 +11,5 @@
         <origin xyz="0 0 0" rpy="0 0 0" />
         <geometry>
-          <mesh filename="package://dsr_description2/meshes/rg6/visual/base_link.stl" /
+          <mesh filename="package://dsr_description2/meshes/rg6/visual/base_link.stl" />
         </geometry>
         <material name="">
@@ -19,5 +19,5 @@
       <collision>
         <origin xyz="0 0 0" rpy="0 0 0" />
-        <geometry
+        <geometry>
           <mesh filename="package://dsr_description2/meshes/rg6/collision/base_link.stl" />
         </geometry>

Commit message: Update onrobot_rg6.xacro

File: onrobot/onrobot_rg_description/urdf/onrobot_rg6.xacro (robot description, xacro)
@@ -11,5 +11,5 @@
         <origin xyz="0 0 0" rpy="0 0 0" />
         <geometry>
-          <mesh filename="package://onrobot_rg_description/meshes/rg6/visual/base_link.stl" />
+          <mesh filename="package://dsr_description2/meshes/rg6/visual/base_link.stl" />
         </geometry>
         <material name="">
@@ -20,5 +20,5 @@
         <origin xyz="0 0 0" rpy="0 0 0" />
         <geometry>
-          <mesh filename="package://onrobot_rg_description/meshes/rg6/collision/base_link.stl" />
+          <mesh filename="package://dsr_description2/meshes/rg6/collision/base_link.stl" />
         </geometry>
       </collision>
