Commit message: Update onrobot_rg6_model.xacro

File: onrobot/onrobot_rg_description/urdf/onrobot_rg6_model.xacro (robot description, xacro)
@@ -1,5 +1,11 @@
 <?xml version="1.0"?>
-<robot name="onrobot_rg6_model" xmlns:xacro="http://wiki.ros.org/xacro">
-  <xacro:include filename="$(find onrobot_rg_description)/urdf/onrobot_rg6_model_macro.xacro" />
+<robot name="onrobot_rg6_model" xmlns:xacro="http://wiki.ros.org/xacro"
+<xacro:arg name="use_gazebo" default="false"/>
+<xacro:property name="gz" value="$(arg use_gazebo)"/>
+<xacro:include filename="$(find onrobot_rg_description)/urdf/onrobot_rg6_model_macro.xacro" />
+  <xacro:if value="${gz}">
+  <!-- Gazebo-->
+    <xacro:include filename="$(find onrobot_rg_description)/urdf/onrobot_rg6_gazebo.xacro" />
+  </xacro:if>
   <xacro:onrobot_rg6 prefix=""/>
 </robot>

Commit message: Update onrobot_rg6_model.xacro

File: onrobot/onrobot_rg_description/urdf/onrobot_rg6_model.xacro (robot description, xacro)
@@ -1,5 +1,11 @@
 <?xml version="1.0"?>
 <robot name="onrobot_rg6_model" xmlns:xacro="http://wiki.ros.org/xacro">
-  <xacro:include filename="$(find onrobot_rg_description)/urdf/onrobot_rg6_model_macro.xacro" />
+<xacro:arg name="use_gazebo" default="false"/>
+<xacro:property name="gz" value="$(arg use_gazebo)"/>
+<xacro:include filename="$(find onrobot_rg_description)/urdf/onrobot_rg6_model_macro.xacro" />
+  <xacro:if value="${gz}">
+  <!-- Gazebo-->
+    <xacro:include filename="$(find onrobot_rg_description)/urdf/onrobot_rg6_gazebo.xacro" />
+  </xacro:if>
   <xacro:onrobot_rg6 prefix=""/>
 </robot>
