Commit message: Update m1013.gz_ros2_control.xacro

File: dsr_description2/ros2_control/m1013.gz_ros2_control.xacro (robot description, xacro)
@@ -79,4 +79,14 @@
         <state_interface name="velocity"/>
       </joint>
+      <joint name="finger_joint">
+        <command_interface name="position">
+          <param name="min">{-2*pi}</param>
+          <param name="max">{2*pi}</param>
+        </command_interface>
+        <state_interface name="position">
+          <param name="initial_value">0.0</param>
+        </state_interface>
+        <state_interface name="velocity"/>
+      </joint>
     </ros2_control>
   </xacro:macro>

Commit message: Update m1013.gz_ros2_control.xacro

File: dsr_description2/ros2_control/m1013.gz_ros2_control.xacro (robot description, xacro)
@@ -79,4 +79,14 @@
         <state_interface name="velocity"/>
       </joint>
+      <joint name="finger_joint">
+          <command_interface name="position">
+            <param name="min">{-2*pi}</param>
+            <param name="max">{2*pi}</param>
+          </command_interface>
+          <state_interface name="position">
+            <param name="initial_value">0.0</param>
+          </state_interface>
+          <state_interface name="velocity"/>
+        </joint>
     </ros2_control>
   </xacro:macro>

Commit message: Update m1013.gz_ros2_control.xacro

File: dsr_description2/ros2_control/m1013.gz_ros2_control.xacro (robot description, xacro)
@@ -80,13 +80,13 @@
       </joint>
       <joint name="finger_joint">
-          <command_interface name="position">
-            <param name="min">{-2*pi}</param>
-            <param name="max">{2*pi}</param>
-          </command_interface>
-          <state_interface name="position">
-            <param name="initial_value">0.0</param>
-          </state_interface>
-          <state_interface name="velocity"/>
-        </joint>
+        <command_interface name="position">
+          <param name="min">{-2*pi}</param>
+          <param name="max">{2*pi}</param>
+        </command_interface>
+        <state_interface name="position">
+          <param name="initial_value">0.0</param>
+        </state_interface>
+        <state_interface name="velocity"/>
+      </joint>
     </ros2_control>
   </xacro:macro>
