Commit message: Update m1013.ros2_control.xacro

File: dsr_description2/ros2_control/m1013.ros2_control.xacro (robot description, xacro)
@@ -111,4 +111,18 @@
         <state_interface name="velocity"/>
       </joint>
+      <joint name="finger_joint">
+        <command_interface name="position">
+          <param name="min">{-2*pi}</param>
+          <param name="max">{2*pi}</param>
+        </command_interface>
+        <command_interface name="velocity">
+          <param name="min">-3.15</param>
+          <param name="max">3.15</param>
+        </command_interface>
+        <state_interface name="position">
+          <param name="initial_value">0.0</param>
+        </state_interface>
+        <state_interface name="velocity"/>
+      </joint>
     </ros2_control>
   </xacro:macro>

Commit message: Update m1013.ros2_control.xacro

File: dsr_description2/ros2_control/m1013.ros2_control.xacro (robot description, xacro)
@@ -111,4 +111,18 @@
         <state_interface name="velocity"/>
       </joint>
+    <joint name="finger_joint">
+        <command_interface name="position">
+          <param name="min">{-2*pi}</param>
+          <param name="max">{2*pi}</param>
+        </command_interface>
+        <command_interface name="velocity">
+          <param name="min">-3.15</param>
+          <param name="max">3.15</param>
+        </command_interface>
+        <state_interface name="position">
+          <param name="initial_value">0.0</param>
+        </state_interface>
+        <state_interface name="velocity"/>
+      </joint>
     </ros2_control>
   </xacro:macro>

Commit message: Update m1013.ros2_control.xacro

File: dsr_description2/ros2_control/m1013.ros2_control.xacro (robot description, xacro)
@@ -111,18 +111,18 @@
         <state_interface name="velocity"/>
       </joint>
-    <joint name="finger_joint">
-        <command_interface name="position">
-          <param name="min">{-2*pi}</param>
-          <param name="max">{2*pi}</param>
-        </command_interface>
-        <command_interface name="velocity">
-          <param name="min">-3.15</param>
-          <param name="max">3.15</param>
-        </command_interface>
-        <state_interface name="position">
-          <param name="initial_value">0.0</param>
-        </state_interface>
-        <state_interface name="velocity"/>
-      </joint>
+      <joint name="finger_joint">
+          <command_interface name="position">
+            <param name="min">{-2*pi}</param>
+            <param name="max">{2*pi}</param>
+          </command_interface>
+          <command_interface name="velocity">
+            <param name="min">-3.15</param>
+            <param name="max">3.15</param>
+          </command_interface>
+          <state_interface name="position">
+            <param name="initial_value">0.0</param>
+          </state_interface>
+          <state_interface name="velocity"/>
+        </joint>
     </ros2_control>
   </xacro:macro>

Commit message: Update m1013.ros2_control.xacro

File: dsr_description2/ros2_control/m1013.ros2_control.xacro (robot description, xacro)
@@ -112,17 +112,17 @@
       </joint>
       <joint name="finger_joint">
-          <command_interface name="position">
-            <param name="min">{-2*pi}</param>
-            <param name="max">{2*pi}</param>
-          </command_interface>
-          <command_interface name="velocity">
-            <param name="min">-3.15</param>
-            <param name="max">3.15</param>
-          </command_interface>
-          <state_interface name="position">
-            <param name="initial_value">0.0</param>
-          </state_interface>
-          <state_interface name="velocity"/>
-        </joint>
+        <command_interface name="position">
+          <param name="min">{-2*pi}</param>
+          <param name="max">{2*pi}</param>
+        </command_interface>
+        <command_interface name="velocity">
+          <param name="min">-3.15</param>
+          <param name="max">3.15</param>
+        </command_interface>
+        <state_interface name="position">
+          <param name="initial_value">0.0</param>
+        </state_interface>
+        <state_interface name="velocity"/>
+      </joint>
     </ros2_control>
   </xacro:macro>
